Commit message: Update dual-arm MR teleop platform

File: ros_backend1.1/src/ur_hande_description/urdf/ur_hande.urdf.xacro (robot description, xacro)
@@ -35,4 +35,5 @@
   <xacro:arg name="sim_gazebo" default="false"/>
   <xacro:arg name="sim_ignition" default="false"/>
+  <xacro:arg name="include_ground_plane" default="false"/>
   <xacro:arg name="simulation_controllers" default=""/>
   <xacro:arg name="initial_positions_file" default="$(find ur_description)/config/initial_positions.yaml"/>
@@ -41,4 +42,5 @@
   <xacro:property name="is_sim_gazebo" value="$(arg sim_gazebo)"/>
   <xacro:property name="is_sim_ignition" value="$(arg sim_ignition)"/>
+  <xacro:property name="include_ground_plane" value="$(arg include_ground_plane)"/>
   <xacro:property name="is_fake_hardware_requested" value="$(arg use_fake_hardware)"/>
   <xacro:property name="hande_grip_min" value="${-0.025 if (is_sim_gazebo or is_sim_ignition) else 0.0}"/>
@@ -51,5 +53,5 @@
   <xacro:include filename="$(find robotiq_hande_description)/urdf/robotiq_hande_gripper.xacro"/>
   <link name="world"/>
-  <xacro:if value="${is_sim_gazebo or is_sim_ignition}">
+  <xacro:if value="${(is_sim_gazebo or is_sim_ignition) and include_ground_plane}">
     <link name="ground_plane">
       <visual>
@@ -131,4 +133,34 @@
     sim_ignition="${is_sim_ignition}"
     generate_ros2_control_tag="${not (is_sim_gazebo or is_sim_ignition)}"/>
+  <!--
+    Gazebo gripper camera is intentionally disabled for the current MR workflow.
+    The active camera preview/recording path is Unity-side:
+      UnityApp/Assets/Scripts/GripperCameraRecorder.cs
+      Unity scene object: GripperDataCamera
+    Keep this placeholder here instead of deleting the idea entirely. If we
+    later want Gazebo-authoritative camera images, re-enable a sensor mounted
+    on $(arg tf_prefix)robotiq_hande_end or $(arg tf_prefix)tool0, then add the
+    required Gazebo/ROS bridge and documentation for /gripper_camera/* topics.
+    Example shape, currently commented out:
+    <gazebo reference="$(arg tf_prefix)robotiq_hande_end">
+      <sensor name="$(arg tf_prefix)gripper_camera" type="camera">
+        <pose>0 0 0 0 0 0</pose>
+        <topic>/$(arg tf_prefix)gripper_camera/image_raw</topic>
+        <update_rate>15</update_rate>
+        <camera>
+          <horizontal_fov>1.5708</horizontal_fov>
+          <image>
+            <width>640</width>
+            <height>480</height>
+            <format>R8G8B8</format>
+          </image>
+          <clip>
+            <near>0.02</near>
+            <far>5.0</far>
+          </clip>
+        </camera>
+      </sensor>
+    </gazebo>
+  -->
   <xacro:if value="${is_sim_gazebo or is_sim_ignition}">
     <!--

File: ros_backend1.1/src/ur_moveit_config/srdf/ur_macro.srdf.xacro (robot description, xacro)
@@ -47,4 +47,39 @@
     <disable_collisions link1="${prefix}tool0" link2="${prefix}wrist_2_link" reason="Never" />
     <disable_collisions link1="${prefix}tool0" link2="${prefix}wrist_3_link" reason="Adjacent" />
+    <disable_collisions link1="${prefix}robotiq_hande_coupler" link2="${prefix}wrist_3_link" reason="Adjacent" />
+    <disable_collisions link1="${prefix}robotiq_hande_coupler" link2="${prefix}tool0" reason="Adjacent" />
+    <disable_collisions link1="${prefix}robotiq_hande_coupler" link2="${prefix}robotiq_hande_link" reason="Adjacent" />
+    <disable_collisions link1="${prefix}robotiq_hande_link" link2="${prefix}tool0" reason="Adjacent" />
+    <disable_collisions link1="${prefix}robotiq_hande_link" link2="${prefix}wrist_3_link" reason="Never" />
+    <!-- Hand-E internal/tool adjacency. These links are part of the gripper assembly and can otherwise create false Servo self-collision reports in normal open/closed poses. -->
+    <disable_collisions link1="${prefix}robotiq_hande_left_finger" link2="${prefix}robotiq_hande_right_finger" reason="Adjacent" />
+    <disable_collisions link1="${prefix}robotiq_hande_left_finger" link2="${prefix}robotiq_hande_link" reason="Adjacent" />
+    <disable_collisions link1="${prefix}robotiq_hande_right_finger" link2="${prefix}robotiq_hande_link" reason="Adjacent" />
+    <disable_collisions link1="${prefix}robotiq_hande_left_finger" link2="${prefix}robotiq_hande_coupler" reason="Never" />
+    <disable_collisions link1="${prefix}robotiq_hande_right_finger" link2="${prefix}robotiq_hande_coupler" reason="Never" />
+    <disable_collisions link1="${prefix}robotiq_hande_left_finger" link2="${prefix}tool0" reason="Never" />
+    <disable_collisions link1="${prefix}robotiq_hande_right_finger" link2="${prefix}tool0" reason="Never" />
+    <!-- The Hand-E is bolted to the UR wrist flange. Its simplified collision
+         cylinders/boxes sit inside the wrist clearance envelope, so Servo can
+         falsely slow down against the compact wrist links even when the visual
+         robot is clear. -->
+    <disable_collisions link1="${prefix}robotiq_hande_coupler" link2="${prefix}wrist_1_link" reason="Adjacent" />
+    <disable_collisions link1="${prefix}robotiq_hande_link" link2="${prefix}wrist_1_link" reason="Adjacent" />
+    <disable_collisions link1="${prefix}robotiq_hande_left_finger" link2="${prefix}wrist_1_link" reason="Adjacent" />
+    <disable_collisions link1="${prefix}robotiq_hande_right_finger" link2="${prefix}wrist_1_link" reason="Adjacent" />
+    <disable_collisions link1="${prefix}robotiq_hande_coupler" link2="${prefix}wrist_2_link" reason="Adjacent" />
+    <disable_collisions link1="${prefix}robotiq_hande_link" link2="${prefix}wrist_2_link" reason="Adjacent" />
+    <disable_collisions link1="${prefix}robotiq_hande_left_finger" link2="${prefix}wrist_2_link" reason="Adjacent" />
+    <disable_collisions link1="${prefix}robotiq_hande_right_finger" link2="${prefix}wrist_2_link" reason="Adjacent" />
+    <disable_collisions link1="${prefix}robotiq_hande_left_finger" link2="${prefix}wrist_3_link" reason="Never" />
+    <disable_collisions link1="${prefix}robotiq_hande_right_finger" link2="${prefix}wrist_3_link" reason="Never" />
+    <disable_collisions link1="${prefix}robotiq_hande_end" link2="${prefix}robotiq_hande_link" reason="Adjacent" />
+    <disable_collisions link1="${prefix}robotiq_hande_end" link2="${prefix}robotiq_hande_coupler" reason="Never" />
+    <disable_collisions link1="${prefix}robotiq_hande_end" link2="${prefix}robotiq_hande_left_finger" reason="Adjacent" />
+    <disable_collisions link1="${prefix}robotiq_hande_end" link2="${prefix}robotiq_hande_right_finger" reason="Adjacent" />
+    <disable_collisions link1="${prefix}robotiq_hande_end" link2="${prefix}tool0" reason="Never" />
+    <disable_collisions link1="${prefix}robotiq_hande_end" link2="${prefix}wrist_1_link" reason="Adjacent" />
+    <disable_collisions link1="${prefix}robotiq_hande_end" link2="${prefix}wrist_2_link" reason="Adjacent" />
+    <disable_collisions link1="${prefix}robotiq_hande_end" link2="${prefix}wrist_3_link" reason="Never" />
     <disable_collisions link1="${prefix}forearm_link" link2="${prefix}upper_arm_link" reason="Adjacent" />
     <disable_collisions link1="${prefix}forearm_link" link2="${prefix}wrist_1_link" reason="Adjacent" />
